File: FeatherWing-switcher/feather-power-supply-sw-smd.kicad_pcb (KiCad board)
At the start: 2 copper layers, 9 parts, among them J4 QWIIC, J5 0.1, Q1 Q_PMOS_GSD

Commit message: update board to version 2
Parts:
- removed TP1: TestPoint, TestPoint:TestPoint_Pad_D1.5mm
- added H4: MountingHole, MountingHole:MountingHole_2.7mm_M2.5, F.Cu at (130.8, 107.0)
- moved J4 10.5 mm to (139.7, 106.7), turned to 0 degrees
- moved J5 8.36 mm to (135.9, 98.9), turned to 90 degrees
- moved REF** 1.98 mm to (138.7, 83.8)
Connections:
- net /SCL renamed SCL
- net /SDA renamed SDA
